File: KicadFiles/R13-BW/R13-BW.kicad_pcb (KiCad board)
At the start: 2 copper layers, 245 x 75 mm, 144 parts, among them J1 Conn_01x01_Pin, J2 Conn_01x04_MountingPin, J3 Conn_01x04_MountingPin, SW1 SW_DPST_x2, SW2 SW_DPST_x2, U1 TPD4E05U06DQAR, U2 STM32F072CBTx, U3 XC6206PxxxMR

Commit message: Add junctions and wires to R13-BW schematic for improved connectivity
- Added a junction at (300.99, 62.23) to enhance signal routing.
- Introduced a junction at (306.07, 67.31) for better circuit integration.
- Removed unnecessary junction at (299.72, 44.45) to clean up the schematic.
- Updated wire connections to reflect new junction placements and maintain circuit integrity.
Parts:
- removed D50, D53: 1N4148WS, My-Fi Footprints:D_SOD-323_HandSoldering
- moved D12 17.0 mm to (239.9, 29.7)
- moved D41 8.28 mm to (230.7, 67.8), turned to 90 degrees
- moved D45 5.00 mm to (256.6, 67.8)
- moved D25 4.00 mm to (233.8, 48.8)
- moved D55 4.00 mm to (192.8, 86.9)
- moved D43 3.00 mm to (242.0, 67.8)
- moved D26 2.00 mm to (247.7, 48.8)
- moved D51 2.00 mm to (124.9, 86.9)
- moved C6 1.37 mm to (49.9, 52.3)
- moved C7 1.37 mm to (50.9, 52.3)
- moved D29 1.00 mm to (34.4, 67.8)
Connections:
- MX13 pad 2: Net-(D12-A) -> Net-(D26-A)
- MX50 pad 2: Net-(D50-A) -> Net-(D51-A)
- MX51 pad 1: Col5 -> Col4
- MX52 pad 1: Col6 -> Col5
- MX53 pad 2: Net-(D53-A) -> Net-(D54-A)
- MX54 pad 1: Col8 -> Col7
- MX55 pad 1: Col9 -> Col8
- MX56 pad 1: Col10 -> Col9
- MX57 pad 1: Col11 -> Col10
Routing:
- net Col11: track 9.53 -> 250.1 mm
- net Row3: track 0.00 -> 232.1 mm
- net Col10: track 0.00 -> 231.6 mm
- net Col12: track 0.00 -> 226.3 mm
- net Row2: track 0.00 -> 225.1 mm, vias 0 -> 2
- net Row1: track 0.00 -> 215.1 mm, vias 0 -> 3
- net Row0: track 0.00 -> 211.5 mm
- net Col9: track 0.00 -> 209.4 mm
- net Col8: track 0.00 -> 186.6 mm
- net Col7: track 0.00 -> 178.9 mm
- net Col5: track 0.00 -> 133.7 mm
- net Col6: track 0.00 -> 125.8 mm
- net Col4: track 0.00 -> 117.3 mm
- net Col3: track 0.00 -> 86.0 mm
- net Col1: track 0.00 -> 84.6 mm
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
Commit message: Implement feature X to enhance user experience and optimize performance
Routing:
- net LED4: track 0.00 -> 48.7 mm, vias 0 -> 2
- net LED3: track 0.00 -> 28.2 mm, vias 0 -> 2
- net LED2: track 0.00 -> 26.7 mm
- net LED_CAPS: track 0.00 -> 25.0 mm
- net LED1: track 0.00 -> 22.6 mm
- net Net-(LED5-A): track 6.72 -> 8.95 mm
- net BOOT-1: track 59.7 -> 60.5 mm

Commit message: Update design rules and add global labels in schematic
- Changed design rule for "courtyards_overlap" from "error" to "ignore".
- Updated hole clearance and hole to hole rules to "ignore".
- Set several silk layer rules to "ignore" to reduce warnings.
- Added multiple global labels in the schematic for better intersheet referencing, including "Col0", "Col1", "Col2", "Col3", "Col4", "Col5", "Col6", "Col7", "Col8", "Col9", "Col10", "Col11", "Col12", "Row0", "Row1", "Row2", and "Row3".
Connections:
- U2 pad 10: unconnected-(U2-PA0-Pad10) -> Col0
- U2 pad 11: unconnected-(U2-PA1-Pad11) -> Row1
- U2 pad 12: unconnected-(U2-PA2-Pad12) -> Row2
- U2 pad 13: unconnected-(U2-PA3-Pad13) -> Row3
- U2 pad 2: unconnected-(U2-PC13-Pad2) -> Col7
- U2 pad 20: unconnected-(U2-PB2-Pad20) -> Row0
- U2 pad 3: unconnected-(U2-PC14-Pad3) -> Col6
- U2 pad 34: unconnected-(U2-PA13-Pad34) -> Col2
- U2 pad 37: unconnected-(U2-PA14-Pad37) -> Col1
- U2 pad 38: unconnected-(U2-PA15-Pad38) -> Col12
- U2 pad 39: unconnected-(U2-PB3-Pad39) -> Col11
- U2 pad 4: unconnected-(U2-PC15-Pad4) -> Col5
- U2 pad 40: unconnected-(U2-PB4-Pad40) -> Col10
- U2 pad 45: unconnected-(U2-PB8-Pad45) -> Col9
- U2 pad 46: unconnected-(U2-PB9-Pad46) -> Col8
- U2 pad 5: unconnected-(U2-PF0-Pad5) -> Col4
- U2 pad 6: unconnected-(U2-PF1-Pad6) -> Col3
Routing:
- net Row3: track 232.1 -> 305.1 mm, vias 0 -> 2
- net Row2: track 225.1 -> 282.5 mm, vias 2 -> 4
- net Col0: track 72.0 -> 107.0 mm, vias 0 -> 2
- net Col3: track 86.0 -> 116.0 mm, vias 0 -> 2
- net Col4: track 117.3 -> 145.3 mm, vias 0 -> 2
- net Col2: track 64.1 -> 91.4 mm, vias 0 -> 1
- net Col5: track 133.7 -> 159.9 mm, vias 0 -> 2
- net Col6: track 125.8 -> 149.9 mm, vias 0 -> 2
- net Col7: track 178.9 -> 201.1 mm, vias 0 -> 2
- net Col8: track 186.6 -> 205.1 mm, vias 0 -> 2
- net Col10: track 231.6 -> 249.8 mm, vias 0 -> 2
- net Col11: track 250.1 -> 267.6 mm, vias 0 -> 2
- net Col12: track 226.3 -> 243.3 mm, vias 0 -> 2
- net Col9: track 209.4 -> 226.3 mm, vias 0 -> 2
- net Row0: track 211.5 -> 227.4 mm, vias 0 -> 2
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- added copper zone on B.Cu, net GND
- added copper zone on F.Cu, net GND
