File: KicadFiles/R13-AW/R13-AW.kicad_pcb (KiCad board)
At the start: 2 copper layers, 245 x 75 mm, 135 parts, among them J1 Conn_01x01_Pin, J2 Conn_01x04_MountingPin, J3 Conn_01x04_MountingPin, SW1 SW_DPST_x2, SW2 SW_DPST_x2, U1 TPD4E05U06DQAR, U2 STM32F072CBTx, U3 XC6206PxxxMR

Commit message: Add junctions and wires to R13-BW schematic for improved connectivity
- Added a junction at (300.99, 62.23) to enhance signal routing.
- Introduced a junction at (306.07, 67.31) for better circuit integration.
- Removed unnecessary junction at (299.72, 44.45) to clean up the schematic.
- Updated wire connections to reflect new junction placements and maintain circuit integrity.
Routing:
- net Col12: track 74.4 -> 272.2 mm
- net Col11: track 41.1 -> 221.2 mm, vias 0 -> 1
- net Col10: track 69.0 -> 239.7 mm
- net Col9: track 64.6 -> 214.4 mm
- net Col8: track 67.1 -> 196.4 mm
- net Col7: track 77.5 -> 186.3 mm
- net Col6: track 44.0 -> 132.4 mm
- net LED2: track 0.00 -> 68.8 mm
- net Col5: track 65.0 -> 132.7 mm
- net LED1: track 0.00 -> 51.3 mm
- net Col4: track 77.6 -> 124.9 mm
- net LED3: track 0.00 -> 38.1 mm, vias 0 -> 2
- net LED4: track 20.5 -> 53.7 mm, vias 0 -> 2
- net Col3: track 66.1 -> 93.3 mm
- net Col2: track 66.6 -> 73.6 mm

Commit message: Update design rules and add global labels in schematic
- Changed design rule settings in R13-AW.kicad_pro to ignore several warnings and errors, including courtyard overlaps, hole clearance, silk edge clearance, and solder mask bridges.
- Added multiple global labels in R13-AW.kicad_sch for better intersheet referencing, including Col0, Col1, Col2, Col3, Col4, Col5, Col6, Col7, Col8, Col9, Col10, Col11, Col12, Row0, Row1, Row2, and Row3.
- Ensured proper placement and formatting for new global labels to enhance readability and maintainability of the schematic.
Connections:
- U2 pad 11: unconnected-(U2-PA1-Pad11) -> Row3
- U2 pad 12: unconnected-(U2-PA2-Pad12) -> Row2
- U2 pad 2: unconnected-(U2-PC13-Pad2) -> Col2
- U2 pad 20: unconnected-(U2-PB2-Pad20) -> Row0
- U2 pad 21: unconnected-(U2-PB10-Pad21) -> Row1
- U2 pad 25: unconnected-(U2-PB12-Pad25) -> Col12
- U2 pad 26: unconnected-(U2-PB13-Pad26) -> Col11
- U2 pad 27: unconnected-(U2-PB14-Pad27) -> Col10
- U2 pad 28: unconnected-(U2-PB15-Pad28) -> Col9
- U2 pad 29: unconnected-(U2-PA8-Pad29) -> Col8
- U2 pad 3: unconnected-(U2-PC14-Pad3) -> Col1
- U2 pad 30: unconnected-(U2-PA9-Pad30) -> Col7
- U2 pad 31: unconnected-(U2-PA10-Pad31) -> Col6
- U2 pad 37: unconnected-(U2-PA14-Pad37) -> Col5
- U2 pad 4: unconnected-(U2-PC15-Pad4) -> Col0
- U2 pad 45: unconnected-(U2-PB8-Pad45) -> Col4
- U2 pad 46: unconnected-(U2-PB9-Pad46) -> Col3
Routing:
- net Row0: track 238.8 -> 290.1 mm
- net Col3: track 93.3 -> 128.0 mm, vias 0 -> 2
- net Col4: track 124.9 -> 158.8 mm, vias 0 -> 2
- net Col0: track 62.7 -> 92.6 mm, vias 0 -> 2
- net Col2: track 73.6 -> 100.7 mm, vias 0 -> 2
- net Col6: track 132.4 -> 158.9 mm, vias 0 -> 4
- net Col7: track 186.3 -> 212.6 mm, vias 0 -> 4
- net Col8: track 196.4 -> 222.6 mm, vias 0 -> 4
- net Col9: track 214.4 -> 240.6 mm, vias 0 -> 4
- net Col10: track 239.7 -> 265.8 mm, vias 0 -> 4
- net Col11: track 221.2 -> 246.9 mm, vias 1 -> 5
- net Col12: track 272.2 -> 297.6 mm, vias 0 -> 4
- net Col5: track 132.7 -> 154.8 mm
- net GND: track 9.52 -> 26.3 mm, vias 3 -> 20
- net Row1: track 219.1 -> 233.8 mm
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- added copper zone on B.Cu, net GND
- added copper zone on F.Cu, net GND
