File: KicadFiles/R13-AH/R13-AH.kicad_pcb (KiCad board)
At the start: 2 copper layers, 245 x 75 mm, 130 parts, among them J1 Conn_01x01_Pin, J2 Conn_01x04_MountingPin, J3 Conn_01x04_MountingPin, SW1 SW_DPST_x2, SW2 SW_DPST_x2, U1 TPD4E05U06DQAR, U2 STM32F072CBTx, U3 XC6206PxxxMR

Commit message: Add junctions and wires to R13-BW schematic for improved connectivity
- Added a junction at (300.99, 62.23) to enhance signal routing.
- Introduced a junction at (306.07, 67.31) for better circuit integration.
- Removed unnecessary junction at (299.72, 44.45) to clean up the schematic.
- Updated wire connections to reflect new junction placements and maintain circuit integrity.
Routing:
- net Col12: track 53.0 -> 269.1 mm
- net Col11: track 43.2 -> 250.8 mm, vias 0 -> 3
- net Col10: track 70.2 -> 269.2 mm, vias 0 -> 2
- net Col9: track 63.6 -> 240.7 mm, vias 0 -> 2
- net Col8: track 65.5 -> 221.9 mm, vias 0 -> 2
- net Col7: track 44.0 -> 179.7 mm, vias 0 -> 2
- net Col6: track 64.1 -> 178.1 mm, vias 0 -> 2
- net Col5: track 65.0 -> 159.0 mm, vias 0 -> 2
- net Row0: track 231.7 -> 307.3 mm
- net Col4: track 65.0 -> 138.3 mm, vias 0 -> 1
- net LED2: track 0.00 -> 67.9 mm
- net LED4: track 0.00 -> 56.2 mm, vias 0 -> 2
- net LED1: track 0.00 -> 50.0 mm
- net Col3: track 65.7 -> 109.8 mm, vias 0 -> 1
- net LED3: track 0.00 -> 40.1 mm, vias 0 -> 2
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
Commit message: Add global labels for columns and rows in R13-AH schematic
- Introduced new global labels for columns (Col0 to Col12) and rows (Row0 to Row3) in the R13-AH schematic.
- Each label includes properties for intersheet references, font size, justification, and positioning.
- Enhanced organization and readability of the schematic by clearly defining input and output connections.
Parts:
- added REF**: myfi, My-Fi Footprints:Logo-MyFi_Silk, F.Cu at (244.4, 33.5)
Connections:
- U2 pad 10: unconnected-(U2-PA0-Pad10) -> Row3
- U2 pad 11: unconnected-(U2-PA1-Pad11) -> Col1
- U2 pad 12: unconnected-(U2-PA2-Pad12) -> Col0
- U2 pad 13: unconnected-(U2-PA3-Pad13) -> Row2
- U2 pad 2: unconnected-(U2-PC13-Pad2) -> Col2
- U2 pad 21: unconnected-(U2-PB10-Pad21) -> Row0
- U2 pad 22: unconnected-(U2-PB11-Pad22) -> Row1
- U2 pad 25: unconnected-(U2-PB12-Pad25) -> Col11
- U2 pad 26: unconnected-(U2-PB13-Pad26) -> Col10
- U2 pad 27: unconnected-(U2-PB14-Pad27) -> Col9
- U2 pad 28: unconnected-(U2-PB15-Pad28) -> Col8
- U2 pad 29: unconnected-(U2-PA8-Pad29) -> Col7
- U2 pad 3: unconnected-(U2-PC14-Pad3) -> Col3
- U2 pad 30: unconnected-(U2-PA9-Pad30) -> Col6
- U2 pad 31: unconnected-(U2-PA10-Pad31) -> Col5
- U2 pad 34: unconnected-(U2-PA13-Pad34) -> Col12
- U2 pad 4: unconnected-(U2-PC15-Pad4) -> Col4
Routing:
- net Col0: track 42.2 -> 69.0 mm, vias 0 -> 1
- net Row3: track 199.7 -> 219.5 mm, vias 0 -> 2
- net Col4: track 138.3 -> 155.6 mm, vias 1 -> 3
- net Col2: track 79.5 -> 96.1 mm, vias 1 -> 3
- net Col3: track 109.8 -> 126.2 mm, vias 1 -> 3
- net Col1: track 76.7 -> 90.9 mm, vias 0 -> 1
- net GND: track 10.5 -> 22.0 mm, vias 3 -> 15
- net Col6: track 178.1 -> 183.2 mm
- net Col5: track 159.0 -> 163.2 mm
- net Col8: track 221.9 -> 226.0 mm
- net Col7: track 179.7 -> 183.8 mm
- net Col9: track 240.7 -> 244.4 mm
- net Col10: track 269.2 -> 272.6 mm
- net Col11: track 250.8 -> 253.8 mm
- net Row1: track 232.4 -> 234.8 mm
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- added copper zone on B.Cu, net GND
- added copper zone on F.Cu, net GND
Other:
- board text added: "Boot"
- board text added: "MF40-R13AH"
- board text added: "Reset"

Commit message: Update DRC exclusions and modify error handling in R13-AH.kicad_pro
- Added multiple DRC exclusions for specific footprints and hole clearances.
- Changed DRC error handling settings for courtyards overlap, hole to hole, nonmirrored text on back layer, silk edge clearance, silk over copper, and silk overlap to "ignore".
- Updated solder mask to copper clearance from 0.0 to 0.005.
Routing:
- net Col0: track 69.0 -> 67.9 mm
- net GND: vias 15 -> 18
